File: SCH16TBreakout.kicad_pcb (KiCad board)
At the start: 2 copper layers, 25.4 x 22.9 mm, 22 parts, among them J1 Conn_01x06, J2 Conn_01x06, U1 SCH16T-K01-1

Commit message: v1.0 finalized
Routing:
- net +3V3: track 48.3 -> 50.1 mm
- net GND: vias 9 -> 16
Other:
- board text added: "SCH16T-K01 IMU"
- board text removed: "SCH16-K01 IMU"
Changed lines of the file:
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@@
 			(outputformat 1)
 			(mirror no)
-			(drillshape 1)
+			(drillshape 0)
 			(scaleselection 1)
-			(outputdirectory "")
+			(outputdirectory "gebers/")
 		)
 	)
@@
 		)
 	)
+	(gr_text "3V3"
+		(at 28.4 56.3 0)
+		(layer "B.SilkS")
+		(effects
+			(font
+				(size 1 1)
+				(thickness 0.15)
+			)
+			(justify left bottom mirror)
+		)
+	)
 	(gr_text "DI"
 		(at 40.3 53.6 0)
@@
 		)
 	)
-	(gr_text "SCH16-K01 IMU\n"
+	(gr_text "SCH16T-K01 IMU\n"
 		(at 43.6 62.2 0)
 		(layer "B.SilkS")
@@
 	)
 	(via
+		(at 41.9 65)
+		(size 0.6)
+		(drill 0.3)
+		(layers "F.Cu" "B.Cu")
+		(free yes)
+		(net 1)
+	)
+	(via
+		(at 32.7 66.5)
+		(size 0.6)
+		(drill 0.3)
+		(layers "F.Cu" "B.Cu")
+		(free yes)
+		(net 1)
+	)
+	(via
 		(at 45.4 57)
 		(size 0.6)
@@
 	)
 	(via
+		(at 27.9 57.3)
+		(size 0.6)
+		(drill 0.3)
+		(layers "F.Cu" "B.Cu")
+		(free yes)
+		(net 1)
+	)
+	(via
 		(at 46.9 65.9)
 		(size 0.6)
@@
 	)
 	(via
+		(at 38.9 62.6)
+		(size 0.6)
+		(drill 0.3)
+		(layers "F.Cu" "B.Cu")
+		(free yes)
+		(net 1)
+	)
+	(via
 		(at 28.8 53.7)
 		(size 0.6)
@@
 	)
 	(via
+		(at 37.5 62.4)
+		(size 0.6)
+		(drill 0.3)
+		(layers "F.Cu" "B.Cu")
+		(free yes)
+		(net 1)
+	)
+	(via
+		(at 27.9 58.6)
+		(size 0.6)
+		(drill 0.3)
+		(layers "F.Cu" "B.Cu")
+		(free yes)
+		(net 1)
+	)
+	(via
 		(at 23.8 58)
 		(size 0.6)
@@
 		(net 1)
 	)
+	(via
+		(at 24.5 63.4)
+		(size 0.6)
+		(drill 0.3)
+		(layers "F.Cu" "B.Cu")
+		(free yes)
+		(net 1)
+	)
 	(segment
 		(start 26.875 60.8)
@@
 	)
 	(segment
-		(start 25.8 55.1)
+		(start 29 55.1)
 		(end 24 55.1)
 		(width 0.2)
@@
 	(segment
 		(start 29.75 59.05)
-		(end 25.8 55.1)
+		(end 29.75 55.85)
 		(width 0.2)
 		(layer "B.Cu")
@@
 	)
 	(segment
+		(start 29.75 55.85)
+		(end 29 55.1)
+		(width 0.2)
+		(layer "B.Cu")
+		(net 2)
+	)
+	(segment
 		(start 34.625 55.7)
 		(end 34.625 57.675)
@@
 	)
 	(segment
-		(start 29.345 56.7)
-		(end 29.445 56.8)
+		(start 29.445 56.8)
+		(end 30.7 56.8)
 		(width 0.2)
 		(layer "F.Cu")
@@
 	)
 	(segment
-		(start 29.445 56.8)
-		(end 30.58 56.8)
+		(start 31.75 55.75)
+		(end 31.75 50.8)
 		(width 0.2)
 		(layer "F.Cu")
@@
 	)
 	(segment
-		(start 30.58 56.8)
-		(end 31.75 55.63)
+		(start 29.345 56.7)
+		(end 29.445 56.8)
 		(width 0.2)
 		(layer "F.Cu")
@@
 	)
 	(segment
-		(start 26.55 56.7)
-		(end 29.345 56.7)
+		(start 30.7 56.8)
+		(end 31.75 55.75)
 		(width 0.2)
 		(layer "F.Cu")
@@
 	)
 	(segment
-		(start 31.75 55.63)
-		(end 31.75 50.8)
+		(start 26.55 56.7)
+		(end 29.345 56.7)
 		(width 0.2)
 		(layer "F.Cu")
@@
 	)
 	(segment
-		(start 34.289999 54.110001)
-		(end 30.8 57.6)
+		(start 26.751 57.999)
+		(end 26.55 58.2)
 		(width 0.2)
 		(layer "F.Cu")
@@
 	)
 	(segment
-		(start 34.289999 50.8)
-		(end 34.289999 54.110001)
+		(start 28.050943 57.999)
+		(end 26.751 57.999)
+		(width 0.2)
+		(layer "F.Cu")
+		(net 9)
+	)
+	(segment
+		(start 31.4649 57.6)
+		(end 29.445 57.6)
 		(width 0.2)
 		(layer "F.Cu")
@@
 	(segment
 		(start 29.445 57.6)
-		(end 27.15 57.6)
+		(end 28.449943 57.6)
 		(width 0.2)
 		(layer "F.Cu")
@@
 	)
 	(segment
-		(start 30.8 57.6)
-		(end 29.445 57.6)
+		(start 34.289999 50.8)
+		(end 34.289999 54.774901)
 		(width 0.2)
 		(layer "F.Cu")
@@
 	)
 	(segment
-		(start 27.15 57.6)
-		(end 26.55 58.2)
+		(start 34.289999 54.774901)
+		(end 31.4649 57.6)
+		(width 0.2)
+		(layer "F.Cu")
+		(net 9)
+	)
+	(segment
+		(start 28.449943 57.6)
+		(end 28.050943 57.999)
 		(width 0.2)
 		(layer "F.Cu")
@@
 	)
 	(segment
-		(start 38.2 65.1)
-		(end 38.2 60.84)
+		(start 38.2 60.7671)
+		(end 40.5671 58.4)
 		(width 0.2)
 		(layer "F.Cu")
@@
 	)
 	(segment
-		(start 40.64 58.4)
+		(start 40.5671 58.4)
 		(end 41.775 58.4)
 		(width 0.2)
@@
 	)
 	(segment
-		(start 38.2 60.84)
-		(end 40.64 58.4)
+		(start 38.2 65.1)
+		(end 38.2 60.7671)
 		(width 0.2)
 		(layer "F.Cu")
@@
 	)
 	(segment
-		(start 36.830001 61.409999)
-		(end 40.64 57.6)
+		(start 40.8 57.6)
+		(end 41.775 57.6)
 		(width 0.2)
 		(layer "F.Cu")
@@
 	)
 	(segment
-		(start 40.64 57.6)
-		(end 41.775 57.6)
+		(start 36.830001 61.569999)
+		(end 40.8 57.6)
 		(width 0.2)
 		(layer "F.Cu")
@@
 	(segment
 		(start 36.830001 68.58)
-		(end 36.830001 61.409999)
+		(end 36.830001 61.569999)
 		(width 0.2)
 		(layer "F.Cu")
@@
 	)
 	(segment
-		(start 39.37 60.33)
-		(end 40.5 59.2)
+		(start 39.37 68.58)
+		(end 39.5 68.45)
 		(width 0.2)
 		(layer "F.Cu")
@@
 	)
 	(segment
-		(start 39.37 68.58)
-		(end 39.37 60.33)
+		(start 39.5 68.45)
+		(end 39.5 60.0342)
 		(width 0.2)
 		(layer "F.Cu")
@@
 	)
 	(segment
-		(start 40.5 59.2)
+		(start 40.3342 59.2)
 		(end 41.775 59.2)
 		(width 0.2)
 		(layer "F.Cu")
+		(net 15)
+	)
+	(segment
+		(start 39.5 60.0342)
+		(end 40.3342 59.2)
+		(width 0.2)
+		(layer "F.Cu")
